Commit message: ratze description
Signed-off-by: lexciese <falahnzk.dev@gmail.com>

File: urdf/ratze.urdf (robot description, URDF)
Before this commit: robot ratze, 13 links, 12 joints
Links:
- link base_link: geometry collision box size=0.26612 0.18000 0.12550; visual mesh filename=package://ratze_description/meshes/stl/base.007.stl scale=1.00000 1.00000 1.00000
- link motor_1: geometry collision cylinder length=0.03175 radius=0.03400; visual mesh filename=package://ratze_description/meshes/stl/Cylinder.stl scale=0.84999 0.84999 0.10948
- link motor_2: geometry collision cylinder length=0.03175 radius=0.03400; visual mesh filename=package://ratze_description/meshes/stl/Cylinder.001.stl scale=0.84999 0.84999 0.10948
- link motor_3: geometry collision cylinder length=0.03175 radius=0.03400; visual mesh filename=package://ratze_description/meshes/stl/Cylinder.003.stl scale=0.84999 0.84999 0.10948
- link motor_4: geometry collision cylinder length=0.03175 radius=0.03400; visual mesh filename=package://ratze_description/meshes/stl/Cylinder.002.stl scale=0.84999 0.84999 0.10948

Commit message: ratze description
Signed-off-by: lexciese <falahnzk.dev@gmail.com>

File: urdf/ratze.urdf (robot description, URDF)
Before this commit: robot ratze, 13 links, 12 joints
Links:
- link motor_1: geometry collision cylinder length=0.03175 radius=0.03400; visual mesh filename=package://ratze_description/meshes/stl/Cylinder.stl scale=1.00000 1.00000 1.00000
- link motor_2: geometry collision cylinder length=0.03175 radius=0.03400; visual mesh filename=package://ratze_description/meshes/stl/Cylinder.001.stl scale=1.00000 1.00000 1.00000
- link motor_3: geometry collision cylinder length=0.03175 radius=0.03400; visual mesh filename=package://ratze_description/meshes/stl/Cylinder.003.stl scale=1.00000 1.00000 1.00000
- link motor_4: geometry collision cylinder length=0.03175 radius=0.03400; visual mesh filename=package://ratze_description/meshes/stl/Cylinder.002.stl scale=1.00000 1.00000 1.00000
Joints:
- joint base_link_joint: origin xyz=-0.00000 0.00000 0.00000 rpy=0.00000 0.00000 0.00000 -> xyz=-0.00000 0.00000 0.01363 rpy=0.00000 0.00000 0.00000
